Commit message: cleaned scripts from unnecessary dependancies

File: src/betabot/betabot_description/urdf/betabot.gazebo.xacro (robot description, xacro)
@@ -97,14 +97,4 @@
     </plugin>
   </gazebo>
-<!-- UNCOMMENT TO FORCE SPECIFIC MESH COLOR FOR BETABOT PARTS  -->
-  <!-- <gazebo reference="base_link">
-    <material>Gazebo/Orange</material>
-  </gazebo>
-  <gazebo reference="left_wheel">
-    <material>Gazebo/Blue</material>
-  </gazebo>
-  <gazebo reference="right_wheel">
-    <material>Gazebo/Blue</material>
-  </gazebo> -->
   <!-- Rplidar -->
   <gazebo reference="rplidar_link">
@@ -151,5 +141,5 @@
       <serviceName>imu_service</serviceName>
       <gaussianNoise>0.0</gaussianNoise>
-      <updateRate>30</updateRate>
+      <updateRate>80</updateRate>
       <imu>
         <noise>
