Commit message: rotated the laser scanner and modified transformation information

File: src/betabot/betabot_description/urdf/betabot.urdf.xacro (robot description, xacro)
@@ -312,5 +312,5 @@
   <joint name="rplidar_joint" type="fixed">
     <axis xyz="0 1 0" />
-    <origin xyz="0 0 .109" rpy="0 0 0"/>
+    <origin xyz="0 0 .109" rpy="0 0 1.57"/>
     <parent link="base_link"/>
     <child link="rplidar_link"/>
